Commit message: fix odin点云坐标系

File: src/rm_simulation/pb_rm_simulation/urdf/odin1_robot.xacro (robot description, xacro)
@@ -179,4 +179,11 @@
     <origin xyz="0.15 0 0.1" rpy="0 0 0"/>
   </joint>
+  <!-- ROS optical convention (Z forward, X right, Y down). -->
+  <link name="tof_optical_frame"/>
+  <joint name="tof_optical_joint" type="fixed">
+    <parent link="tof_link"/>
+    <child link="tof_optical_frame"/>
+    <origin xyz="0 0 0" rpy="${-PI/2} 0 ${-PI/2}"/>
+  </joint>
   <!-- rgb_cameral-->
   <link name="rgb_camera_link">
@@ -194,4 +201,10 @@
     <child link="rgb_camera_link"/>
     <origin xyz="0.15 0 0.1" rpy="0 0 0"/>
+  </joint>
+  <link name="rgb_camera_optical_frame"/>
+  <joint name="rgb_camera_optical_joint" type="fixed">
+    <parent link="rgb_camera_link"/>
+    <child link="rgb_camera_optical_frame"/>
+    <origin xyz="0 0 0" rpy="${-PI/2} 0 ${-PI/2}"/>
   </joint>
   <!-- Gazebo插件设置相关 -->
@@ -226,5 +239,5 @@
         </ros>
         <camera_name>depthmod</camera_name>
-        <frame_name>tof_link</frame_name>
+        <frame_name>tof_optical_frame</frame_name>
         <hack_baseline>0.07</hack_baseline>
         <min_depth>0.2</min_depth>
@@ -248,5 +261,5 @@
         </ros>
         <camera_name>rgbcamera</camera_name>
-        <frame_name>rgb_camera_link</frame_name>
+        <frame_name>rgb_camera_optical_frame</frame_name>
       </plugin>
     </sensor>
